Commit message: ...

File: assets/ros-package-sets/abb-noetic-devel/abb_irb1200_support/urdf/irb1200_7_70_macro.xacro (robot description, xacro)
@@ -130,5 +130,5 @@
     </joint>
     <joint type="revolute" name="${prefix}joint_5">
-      <origin xyz="0.351 0 0 " rpy="0 0 0"/>
+      <origin xyz="0.451 0 0 " rpy="0 0 0"/>
       <axis xyz="0 1 0"/>
       <parent link="${prefix}link_4"/>

File: assets/ros-package-sets/abb-noetic-devel/abb_irb52_support/urdf/irb52_7_120_macro.xacro (robot description, xacro)
@@ -146,5 +146,5 @@
     </joint>
     <joint name="${prefix}joint_5" type="revolute">
-      <origin xyz="0.600 0 0" rpy="0 0 0"/>
+      <origin xyz="0.000 0 0" rpy="0 0 0"/>
       <parent link="${prefix}link_4"/>
       <child link="${prefix}link_5"/>

File: assets/ros-package-sets/abb-noetic-devel/abb_irb52_support/urdf/irb52_7_145_macro.xacro (robot description, xacro)
@@ -146,5 +146,5 @@
     </joint>
     <joint name="${prefix}joint_5" type="revolute">
-      <origin xyz="0.600 0 0" rpy="0 0 0"/>
+      <origin xyz="0.000 0 0" rpy="0 0 0"/>
       <parent link="${prefix}link_4"/>
       <child link="${prefix}link_5"/>
